File: Hardware/untitled.brd (EAGLE design)
At the start: 44.1 x 26.7 mm, 19 parts, among them Q1 2N3904, Q2 2N3904

Commit message: Old board cleanup
Parts:
- moved BACK 2.54 mm to (39.4, 15.2)
- moved CENTER 2.54 mm to (39.4, 21.6)
- moved FRONT 2.54 mm to (39.4, 8.89)
- moved R7 2.54 mm to (38.1, 24.8)
- moved D2 1.91 mm to (5.71, 15.2)
- moved BACK_FAN 1.27 mm to (11.4, 24.1), turned to 270 degrees
- moved FRONT_FAN 1.27 mm to (27.9, 24.1), turned to 270 degrees
Routing:
- net 5V: track 0.00 -> 96.1 mm
- net 3.3V: track 28.0 -> 25.4 mm
- net GND: track 66.6 -> 64.0 mm
- net N$3: track 25.4 -> 23.7 mm
- net GPIO4: track 34.0 -> 35.4 mm
- removed copper zone on layer 16, net 5V
Other:
- board size 44.1 x 26.7 mm -> 42.9 x 26.7 mm
- board text added: "+"
- board text added: "-"
